File: MCPGrundplatte_16_Ausgabe.brd (EAGLE design)
At the start: 49.2 x 80 mm, 36 parts, among them IC1 ULN2803, IC2 74HC14N, IC3 74HC14N, X1GPA0-7 MKDSN1,5/9-5,08, X2 MKDSN1,5/2-5,08, X2GPB0-7 MKDSN1,5/9-5,08

Commit message: Neuen 16 Fach Output und 8In8Out hinzugefügt
Parts:
- removed C1: 100Nf, rcl:C025-024X044
- removed C11, C3, C4, C5, C6, C7, C8: 100nF, rcl:C025-024X044
- removed IC2, IC3: 74HC14N, 74xx-eu:DIL14
- removed R1, R10, R11, R12, R13, R14, R15, R16, R2, R3, R4, R5, R6, R7, R8, R9: 10k, rcl:0207/10
- removed RN2: 100K, resistor-net:RN-9
- added IC6: ULN2803, uln-udn:DIL18
- moved C19 25.1 mm to (11.4, 15.2), turned to 270 degrees
- moved C20 24.4 mm to (38.1, 63.5)
Connections:
- removed net GPB0: R7.1, R8.2, X2GPB0-7.9
- removed net GPB1: R4.1, R5.1, X2GPB0-7.8
- removed net GPB2: R1.1, R3.2, X2GPB0-7.7
- removed net GPB3: R2.2, R6.1, X2GPB0-7.6
- removed net GPB4: R12.1, R9.2, X2GPB0-7.5
- removed net GPB5: R10.1, R11.2, X2GPB0-7.4
- removed net GPB6: R15.2, R16.1, X2GPB0-7.3
- removed net GPB7: R13.1, R14.2, X2GPB0-7.2
- removed net N$11: C11.1, IC3.1, R13.2
- removed net N$2: C7.1, IC2.5, R1.2
- removed net N$4: C1.1, IC2.13, R6.2
- removed net N$5: C6.1, IC2.3, R4.2
- removed net N$6: C5.1, IC2.1, R7.2
- removed net N$7: C4.1, IC2.9, R10.2
- removed net N$8: C3.1, IC2.11, R12.2
- removed net N$9: C8.1, IC3.13, R16.2
- new net IC6_OUT1: IC6.18, X2GPB0-7.9
- new net IC6_OUT2: IC6.17, X2GPB0-7.8
- new net IC6_OUT3: IC6.16, X2GPB0-7.7
- new net IC6_OUT4: IC6.15, X2GPB0-7.6
- new net IC6_OUT5: IC6.14, X2GPB0-7.5
- new net IC6_OUT6: IC6.13, X2GPB0-7.4
- new net IC6_OUT7: IC6.12, X2GPB0-7.3
- new net IC6_OUT8: IC6.11, X2GPB0-7.2
- net +12V: now also C19.2, C20.1, IC6.10, X2GPB0-7.1
- net GND: now also IC6.9; no longer C1.2, C11.2, C3.2, C4.2, C5.2, C6.2, C7.2, C8.2, IC2.7, IC3.10, IC3.11, IC3.3, IC3.4, IC3.5, IC3.6, IC3.7, IC3.8, IC3.9, X2GPB0-7.1
- net GPB0.: now also IC6.1; no longer IC2.2, RN2.9
- net GPB1.: now also IC6.2; no longer IC2.4, RN2.8
- net GPB2.: now also IC6.3; no longer IC2.6, RN2.7
- net GPB3.: now also IC6.4; no longer IC2.12, RN2.6
- net GPB4.: now also IC6.5; no longer IC2.10, RN2.5
- net GPB5.: now also IC6.6; no longer IC2.8, RN2.4
- net GPB6.: now also IC6.7; no longer IC3.12, RN2.3
- net GPB7.: now also IC6.8; no longer IC3.2, RN2.2
- net VDD: no longer C19.2, C20.1, IC2.14, IC3.14, R11.1, R14.1, R15.1, R2.1, R3.1, R5.2, R8.1, R9.1, RN2.1
Routing:
- net VDD: track 146.5 -> 62.1 mm
- net +12V: track 71.9 -> 140.2 mm
- net N$9: track 30.5 -> 0.00 mm
- net N$11: track 26.1 -> 0.00 mm
- net N$5: track 24.0 -> 0.00 mm
- net N$2: track 22.7 -> 0.00 mm
- net N$6: track 19.7 -> 0.00 mm
- net IC6_OUT1: track 0.00 -> 15.1 mm
- net GPB2.: track 23.5 -> 37.2 mm
- net IC6_OUT2: track 0.00 -> 12.5 mm
- net GPB0: track 12.2 -> 0.00 mm
- net GPB1.: track 28.6 -> 40.8 mm
- net IC6_OUT8: track 0.00 -> 11.5 mm
- net IC6_OUT3: track 0.00 -> 11.5 mm
- net IC6_OUT7: track 0.00 -> 10.5 mm
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Other:
- board text added: "SX2MCP23017 16 Output Version V2"
- board text removed: "SX2MCP23017 INPUT Version V5"
