File: MCPGrundplatte/MCPGrundplatte16UniversalInputoutput.sch (EAGLE design)
At the start: 60 parts, among them IC2 74HC14N, IC3 74HC14N, IC4 74HC14N, X1GPA0-7 MKDSN1,5/9-5,08, X2GPB0-7 MKDSN1,5/9-5,08

Commit message: Neu organisiert
Parts:
- removed C15, C16, C17, C18, C21: 100nF, rcl:C-EU025-024X044
- removed R29, R30, R31, R32: 10k, rcl:R-EU_0207/10
- removed RN1: 100K, resistor-net:RN08
- added C2: 100Nf, rcl:C-EU025-024X044
- added C9: 100nF, rcl:C-EU025-024X044
- added IC1: ULN2803, uln-udn:ULN2803A
- added IC5: 74HC14N, 74xx-eu:74HC14N
- added JP1, JP10, JP11, JP12, JP13, JP14, JP15, JP16: (no value), jumper:JP2E
- added SV2: (no value), con-lstb:MA04-2
- added X2: MKDSN1,5/2-5,08, con-phoenix-508:MKDSN1,5/2-5,08
- IC4: value 74HC14N -> ULN2803; device 74xx-eu:74HC14N -> uln-udn:ULN2803A
Connections:
- removed net GPA0: R20.2, R32.1, X1GPA0-7-9.KL
- removed net GPA1: R24.1, R26.2, X1GPA0-7-8.KL
- removed net GPA2.: IC4D.O, RN1.4, SV4.5
- removed net GPA3.: IC4E.O, RN1.5, SV4.6
- removed net GPA4.: IC4F.O, RN1.6, SV4.7
- removed net GPA5: R30.2, R31.1, X1GPA0-7-4.KL
- removed net GPA6: R17.2, R18.1, X1GPA0-7-3.KL
- removed net GPA7: R19.2, R21.1, X1GPA0-7-2.KL
- removed net GPB7: R13.1, R14.2, X2GPB0-7-2.KL
- removed net N$52: C21.1, IC3B.I, R32.2
- new net +12V: IC1.CD+, IC4.CD+, SV2.1, SV2.2, SV2.3, SV2.4, X1GPA0-7-1.KL, X2-1.KL
- new net IC2_OUT1: IC1.O1, X1GPA0-7-9.KL
- new net IC2_OUT2: IC1.O2, X1GPA0-7-8.KL
- new net IC2_OUT3: IC1.O3, X1GPA0-7-7.KL
- new net IC2_OUT4: IC1.O4, X1GPA0-7-6.KL
- new net IC2_OUT5: IC1.O5, X1GPA0-7-5.KL
- new net IC2_OUT6: IC1.O6, X1GPA0-7-4.KL
- new net IC2_OUT7: IC1.O7, X1GPA0-7-3.KL
- new net IC2_OUT8: IC1.O8, X1GPA0-7-2.KL
- new net N$1: IC2A.O, JP13.1
- new net N$14: C2.1, IC5A.I, R28.2
- new net N$15: IC3D.O, JP14.1
- new net N$17: IC4.O8, R13.1, R14.2, X2GPB0-7-2.KL
- new net N$18: IC2F.O, JP11.1
- new net N$19: IC3A.O, JP12.1
- new net N$22: IC4.I5, JP15.3
- new net N$23: C13.1, IC5E.I, R19.2
- new net N$24: IC4.O5, R12.1, R9.2, X2GPB0-7-5.KL
- new net N$25: IC4.I6, JP16.3
- new net N$26: IC4.I7, JP13.3
- new net N$27: IC4.I8, JP14.3
- new net N$29: C12.1, IC5D.I, R21.2
- new net N$3: IC2E.O, JP10.1
- new net N$30: IC2D.O, JP1.1
- new net N$31: C10.1, IC5C.I, R23.2
- new net N$32: C9.1, IC5B.I, R26.2
- new net N$33: IC4.I2, JP10.3
- new net N$34: IC4.I1, JP1.3
- new net N$35: R27.2, R28.1
- new net N$37: R21.1, R22.2
- new net N$43: R25.2, R26.1
- net GND: now also C2.2, C9.2, IC1.GND, IC3B.I, IC3B.O, IC3C.I, IC3C.O, IC4.GND, SV2.5, SV2.6, SV2.7, SV2.8, X2-2.KL; no longer C15.2, C16.2, C17.2, C18.1, C21.2, IC4P.GND, X1GPA0-7-1.KL
- net GPA0.: now also IC1.I1; no longer IC3B.O, RN1.2
- net GPA1.: now also IC1.I2; no longer IC3C.O, RN1.3
- net GPA2: now also IC1.I3, SV4.5; no longer R22.2, R23.1, X1GPA0-7-7.KL
- net GPA3: now also IC1.I4, SV4.6; no longer R25.2, R27.1, X1GPA0-7-6.KL
- net GPA4: now also IC1.I5, SV4.7; no longer R28.2, R29.1, X1GPA0-7-5.KL
- net GPA5.: now also IC1.I6; no longer IC4A.O, RN1.7
- net GPA6.: now also IC1.I7; no longer IC4B.O, RN1.8
- net GPA7.: now also IC1.I8; no longer IC4C.O, RN1.9
- net GPB0: now also IC4.O1
- net GPB0.: now also JP1.2; no longer IC2D.O
- net GPB1: now also IC4.O2
- net GPB1.: now also JP10.2; no longer IC2E.O
- net GPB2: now also IC4.O3
- net GPB2.: now also JP11.2; no longer IC2F.O
- net GPB3: now also R17.2, R18.1; no longer R2.2, R6.1, X2GPB0-7-6.KL
- net GPB3.: now also JP12.2; no longer IC2A.O
- net GPB4: now also R19.1, R20.1; no longer R12.1, R9.2, X2GPB0-7-5.KL
- net GPB4.: now also JP15.2; no longer IC2B.O
- net GPB5: now also IC4.O6
- net GPB5.: now also JP16.2; no longer IC2C.O
- net GPB6: now also R23.1, R24.2; no longer R15.2, R16.1, X2GPB0-7-3.KL
- net GPB6.: now also JP13.2; no longer IC3A.O
- net GPB7.: now also JP14.2; no longer IC3D.O
- net N$10: now also IC4.I3, JP11.3; no longer C10.1, IC3C.I, R24.2
- net N$12: now also IC4.O7, R2.2, R6.1, X2GPB0-7-3.KL; no longer C12.1, IC4E.I, R27.2
- net N$13: now also IC4.I4, JP12.3; no longer C13.1, IC4F.I, R29.2
- net N$16: now also C14.1, IC5F.I; no longer C15.1, IC4B.I
- net N$20: now also IC2B.O, JP15.1; no longer C16.1, IC4C.I, R21.2
- net N$21: now also IC2C.O, JP16.1; no longer C17.1, IC4D.I, R23.2
- net N$28: now also IC4.O4, R15.2, R16.1, X2GPB0-7-6.KL; no longer C14.1, IC4A.I, R31.2
- net VDD: now also R20.2, R24.1; no longer C18.2, IC4P.VCC, R19.1, R20.1, R26.1, R28.1, R30.1, RN1.1
Other:
- moved on the sheet: C1, C10, C11, C12, C13, C14, C3, C4, C5, C6, C7, C8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

Commit message: Neue Hardware
Parts:
- removed R1, R3: 10k, rcl:R-EU_0207/10
- added C15, C16: 100Nf, rcl:C-EU025-024X044
- added C17: 100nF, rcl:C-EU025-024X044
- added JP2, JP3, JP4, JP5, JP6, JP7, JP8, JP9: (no value), jumper:JP2E
- added R29, R30, R31, R32, R33, R34: 10k, rcl:R-EU_0207/2V
- added RN1: 100K, resistor-net:RN08
- R10, R11, R12, R13, R14, R15, R16, R17, R18, R19, R2, R20, R21, R22, R23, R24, R25, R26, R27, R28, R4, R5, R6, R7, R8, R9: device rcl:R-EU_0207/10 -> rcl:R-EU_0207/2V
Connections:
- removed net GPA0.: IC1.I1, SV4.3
- removed net GPA1.: IC1.I2, SV4.4
- removed net GPA5.: IC1.I6, SV4.8
- removed net GPA6.: IC1.I7, SV4.9
- removed net GPA7.: IC1.I8, SV4.10
- removed net IC2_OUT1: IC1.O1, X1GPA0-7-9.KL
- removed net IC2_OUT2: IC1.O2, X1GPA0-7-8.KL
- removed net IC2_OUT3: IC1.O3, X1GPA0-7-7.KL
- removed net IC2_OUT4: IC1.O4, X1GPA0-7-6.KL
- removed net IC2_OUT5: IC1.O5, X1GPA0-7-5.KL
- removed net IC2_OUT6: IC1.O6, X1GPA0-7-4.KL
- removed net IC2_OUT7: IC1.O7, X1GPA0-7-3.KL
- removed net IC2_OUT8: IC1.O8, X1GPA0-7-2.KL
- removed net N$17: IC4.O8, R13.1, R14.2, X2GPB0-7-2.KL
- removed net N$24: IC4.O5, R12.1, R9.2, X2GPB0-7-5.KL
- removed net N$28: IC4.O4, R15.2, R16.1, X2GPB0-7-6.KL
- removed net N$37: R21.1, R22.2
- removed net N$43: R25.2, R26.1
- new net GPA0: IC1.O1, R17.2, R23.2, X1GPA0-7-9.KL
- new net GPA1: IC1.O2, R18.2, R24.2, X1GPA0-7-8.KL
- new net GPA5: IC1.O6, R22.2, R28.2, X1GPA0-7-4.KL
- new net GPA6: IC1.O7, R29.2, R31.2, X1GPA0-7-3.KL
- new net GPA7: IC1.O8, R30.2, R32.2, X1GPA0-7-2.KL
- new net GPB7: IC4.O8, R15.2, R9.2, X2GPB0-7-2.KL
- new net N$36: IC5F.O, JP2.3
- new net N$38: IC5E.O, JP3.3
- new net N$39: IC5D.O, JP4.3
- new net N$40: IC5C.O, JP5.3
- new net N$41: C16.1, IC3E.I, R32.1
- new net N$42: IC3E.O, JP9.3
- new net N$44: JP3.2, RN1.8, SV4.4
- new net N$45: IC5B.O, JP6.3
- new net N$46: IC5A.O, JP7.3
- new net N$47: IC3C.O, JP8.3
- new net N$48: JP5.2, RN1.6, SV4.6
- new net N$49: IC1.I3, JP4.1
- new net N$50: IC1.I1, JP2.1
- new net N$51: IC1.I5, JP6.1
- new net N$52: IC1.I4, JP5.1
- new net N$53: IC1.I2, JP3.1
- new net N$54: JP4.2, RN1.7, SV4.5
- new net N$55: IC1.I7, JP8.1
- new net N$56: IC1.I6, JP7.1
- new net N$57: IC1.I8, JP9.1
- new net N$58: JP6.2, RN1.5, SV4.7
- new net N$59: JP7.2, RN1.4, SV4.8
- new net N$60: JP8.2, RN1.3, SV4.9
- new net N$61: JP9.2, RN1.2, SV4.10
- net GND: now also C15.2, C16.2, C17.2, IC5P.GND; no longer IC3C.I, IC3C.O, IC3E.I, IC3E.O
- net GPA2: now also IC1.O3, R19.2, R25.2, X1GPA0-7-7.KL; no longer IC1.I3, SV4.5
- net GPA3: now also IC1.O4, R20.2, R26.2, X1GPA0-7-6.KL; no longer IC1.I4, SV4.6
- net GPA4: now also IC1.O5, R21.2, R27.2, X1GPA0-7-5.KL; no longer IC1.I5, SV4.7
- net GPB0: now also R10.2, R5.2; no longer R7.1, R8.2
- net GPB1: now also R11.2, R4.2; no longer R4.1, R5.1
- net GPB2: now also R33.2, R34.2; no longer R1.1, R3.2
- net GPB3: now also IC4.O4, R12.2, R16.2, X2GPB0-7-6.KL; no longer R17.2, R18.1
- net GPB4: now also IC4.O5, R14.2, R2.2, X2GPB0-7-5.KL; no longer R19.1, R20.1
- net GPB5: now also R7.2, R8.2; no longer R10.1, R11.2
- net GPB6: now also IC4.O7, R13.2, R6.2, X2GPB0-7-3.KL; no longer R23.1, R24.2
- net N$11: now also R9.1; no longer R13.2
- net N$12: now also JP2.2, RN1.9, SV4.3; no longer IC4.O7, R2.2, R6.1, X2GPB0-7-3.KL
- net N$14: now also R22.1; no longer R28.2
- net N$16: now also R17.1; no longer R18.2
- net N$2: now also R33.1; no longer R1.2
- net N$23: now also R18.1; no longer R19.2
- net N$29: now also R19.1; no longer R21.2
- net N$31: now also R20.1; no longer R23.2
- net N$32: now also R21.1; no longer R26.2
- net N$35: now also C15.1, IC3C.I, R29.1; no longer R27.2, R28.1
- net N$4: now also R6.1; no longer R6.2
- net N$5: now also R4.1; no longer R4.2
- net N$6: now also R5.1; no longer R7.2
- net N$7: now also R7.1; no longer R10.2
- net N$8: now also R2.1; no longer R12.2
- net N$9: now also R12.1; no longer R16.2
- net VDD: now also C17.1, IC5P.VCC, R10.1, R13.1, R16.1, R23.1, R26.1, R27.1, R28.1, R30.1, R31.1, R34.1, RN1.1; no longer R17.1, R2.1, R20.2, R22.1, R3.1, R5.2, R9.1
Other:
- moved on the sheet: C19, C20, IC1, IC2P, IC3P, R10, R11, R12, R13, R14, R15, R16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

Commit message: Neuen OutPut 16x hinzugefügt
Parts:
- removed C1, C15, C16, C2: 100Nf, rcl:C-EU025-024X044
- removed C10, C11, C12, C13, C14, C17, C19, C20, C3, C4, C5, C6, C7, C8, C9: 100nF, rcl:C-EU025-024X044
- removed IC2, IC3, IC5: 74HC14N, 74xx-eu:74HC14N
- removed JP1, JP10, JP11, JP12, JP13, JP14, JP15, JP16, JP2, JP3, JP4, JP5, JP6, JP7, JP8, JP9: (no value), jumper:JP2E
- removed R10, R11, R12, R13, R14, R15, R16, R17, R18, R19, R2, R20, R21, R22, R23, R24, R25, R26, R27, R28, R29, R30, R31, R32, R33, R34, R4, R5, R6, R7, R8, R9: 10k, rcl:R-EU_0207/2V
- removed RN1, RN2: 100K, resistor-net:RN08
Connections:
- removed net N$10: IC4.I3, JP11.3
- removed net N$11: C11.1, IC3D.I, R9.1
- removed net N$12: JP2.2, RN1.9, SV4.3
- removed net N$13: IC4.I4, JP12.3
- removed net N$14: C2.1, IC5A.I, R22.1
- removed net N$15: IC3D.O, JP14.1
- removed net N$16: C14.1, IC5F.I, R17.1
- removed net N$18: IC2F.O, JP11.1
- removed net N$19: IC3A.O, JP12.1
- removed net N$20: IC2B.O, JP15.1
- removed net N$21: IC2C.O, JP16.1
- removed net N$22: IC4.I5, JP15.3
- removed net N$23: C13.1, IC5E.I, R18.1
- removed net N$25: IC4.I6, JP16.3
- removed net N$26: IC4.I7, JP13.3
- removed net N$27: IC4.I8, JP14.3
- removed net N$29: C12.1, IC5D.I, R19.1
- removed net N$30: IC2D.O, JP1.1
- removed net N$31: C10.1, IC5C.I, R20.1
- removed net N$32: C9.1, IC5B.I, R21.1
- removed net N$33: IC4.I2, JP10.3
- removed net N$34: IC4.I1, JP1.3
- removed net N$35: C15.1, IC3C.I, R29.1
- removed net N$36: IC5F.O, JP2.3
- removed net N$38: IC5E.O, JP3.3
- removed net N$39: IC5D.O, JP4.3
- removed net N$40: IC5C.O, JP5.3
- removed net N$41: C16.1, IC3E.I, R32.1
- removed net N$42: IC3E.O, JP9.3
- removed net N$44: JP3.2, RN1.8, SV4.4
- removed net N$45: IC5B.O, JP6.3
- removed net N$46: IC5A.O, JP7.3
- removed net N$47: IC3C.O, JP8.3
- removed net N$48: JP5.2, RN1.6, SV4.6
- removed net N$49: IC1.I3, JP4.1
- removed net N$50: IC1.I1, JP2.1
- removed net N$51: IC1.I5, JP6.1
- removed net N$52: IC1.I4, JP5.1
- removed net N$53: IC1.I2, JP3.1
- removed net N$54: JP4.2, RN1.7, SV4.5
- removed net N$55: IC1.I7, JP8.1
- removed net N$56: IC1.I6, JP7.1
- removed net N$57: IC1.I8, JP9.1
- removed net N$58: JP6.2, RN1.5, SV4.7
- removed net N$59: JP7.2, RN1.4, SV4.8
- removed net N$60: JP8.2, RN1.3, SV4.9
- removed net N$61: JP9.2, RN1.2, SV4.10
- removed net N$9: C8.1, IC3A.I, R12.1
- net GND: no longer C1.2, C10.2, C11.2, C12.2, C13.2, C14.2, C15.2, C16.2, C17.2, C19.1, C2.2, C20.2, C3.2, C4.2, C5.2, C6.2, C7.2, C8.2, C9.2, IC2P.GND, IC3B.I, IC3B.O, IC3F.I, IC3F.O, IC3P.GND, IC5P.GND
- net GPA0: no longer R17.2, R23.2
- net GPA1: no longer R18.2, R24.2
- net GPA2: no longer R19.2, R25.2
- net GPA3: no longer R20.2, R26.2
- net GPA4: no longer R21.2, R27.2
- net GPA5: no longer R22.2, R28.2
- net GPA6: no longer R29.2, R31.2
- net GPA7: no longer R30.2, R32.2
- net GPB0: no longer R10.2, R5.2
- net GPB0.: now also IC4.I1; no longer JP1.2, RN2.9
- net GPB1: no longer R11.2, R4.2
- net GPB1.: now also IC4.I2; no longer JP10.2, RN2.8
- net GPB2: no longer R33.2, R34.2
- net GPB2.: now also IC4.I3; no longer JP11.2, RN2.7
- net GPB3: no longer R12.2, R16.2
- net GPB3.: now also IC4.I4; no longer JP12.2, RN2.6
- net GPB4: no longer R14.2, R2.2
- net GPB4.: now also IC4.I5; no longer JP15.2, RN2.5
- net GPB5: no longer R7.2, R8.2
- net GPB5.: now also IC4.I6; no longer JP16.2, RN2.4
- net GPB6: no longer R13.2, R6.2
- net GPB6.: now also IC4.I7; no longer JP13.2, RN2.3
- net GPB7: no longer R15.2, R9.2
- net GPB7.: now also IC4.I8; no longer JP14.2, RN2.2
- net N$1: now also IC1.I6, SV4.8; no longer IC2A.O, JP13.1
- net N$2: now also IC1.I1, SV4.3; no longer C7.1, IC2F.I, R33.1
- net N$3: now also IC1.I2, SV4.4; no longer IC2E.O, JP10.1
- net N$4: now also IC1.I3, SV4.5; no longer C1.1, IC2A.I, R6.1
- net N$5: now also IC1.I4, SV4.6; no longer C6.1, IC2E.I, R4.1
- net N$6: now also IC1.I5, SV4.7; no longer C5.1, IC2D.I, R5.1
- net N$7: now also IC1.I7, SV4.9; no longer C4.1, IC2C.I, R7.1
- net N$8: now also IC1.I8, SV4.10; no longer C3.1, IC2B.I, R2.1
- net VDD: no longer C17.1, C19.2, C20.1, IC2P.VCC, IC3P.VCC, IC5P.VCC, R10.1, R11.1, R13.1, R14.1, R15.1, R16.1, R23.1, R24.1, R25.1, R26.1, R27.1, R28.1, R30.1, R31.1, R34.1, R8.1, RN1.1, RN2.1
Other:
- moved on the sheet: IC1, SV4, X1GPA0-7-2, X1GPA0-7-3, X1GPA0-7-4, X1GPA0-7-5, X1GPA0-7-6, X1GPA0-7-7, X1GPA0-7-8, X1GPA0-7-9, X2GPB0-7-2, X2GPB0-7-3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
