File: MCP23017_Aufsatz/MCP23017_Aufsatz_Verzweiger_V1.sch (EAGLE design)
At the start: 79 parts, among them IC1 ULN2803, IC2 74HC14N, IC3 74HC14N, IC4 ULN2803, IC5 74HC14N, X1GPA0-7 MKDSN1,5/9-5,08, X2 MKDSN1,5/2-5,08, X2GPB0-7 MKDSN1,5/9-5,08

Commit message: Neue Hardware
Parts:
- removed C1, C15, C16: 100Nf, rcl:C-EU025-024X044
- removed C10, C11, C12, C13, C14, C19, C20, C3, C4, C5, C6, C7, C8, C9: 100nF, rcl:C-EU025-024X044
- removed IC2, IC3, IC5: 74HC14N, 74xx-eu:74HC14N
- removed IC4: ULN2803, uln-udn:ULN2803A
- removed R10, R11, R12, R13, R14, R15, R16, R17, R18, R19, R20, R21, R22, R23, R24, R25, R26, R27, R28, R29, R30, R31, R32, R33, R34, R9: 10k, rcl:R-EU_0207/2V
- removed RN1, RN2: 100K, resistor-net:RN08
- removed X1GPA0-7, X2GPB0-7: MKDSN1,5/9-5,08, con-phoenix-508:MKDSN1,5/9-5,08
- removed X2: MKDSN1,5/2-5,08, con-phoenix-508:MKDSN1,5/2-5,08
- added ADR1: ADR, pinhead:PINHD-2X3
- added JP17, JP18: (no value), jumper:JP2E
- added LED1: Grün, led:LED3MM
- added R3: 1k, rcl:R-EU_0207/10
- added S1: (no value), switch-omron:10-XX
- added SV1: (no value), con-lsta:FE10-1
- C2: value 100Nf -> 100nF; device rcl:C-EU025-024X044 -> rcl:C-EU025-025X050
- IC1: value ULN2803 -> MCP23017SP; device uln-udn:ULN2803A -> microchip:MCP23017SP
- JP1: value (none) -> JP1; device jumper:JP2E -> pinhead:PINHD-2X6/90
- JP2: device jumper:JP2E -> jumper:JP1E
- R2, R8: device rcl:R-EU_0207/2V -> rcl:R-EU_0207/10
- R4, R5: value 10k -> 1k; device rcl:R-EU_0207/2V -> rcl:R-EU_0207/10
- R6, R7: value 10k -> 4,7k; device rcl:R-EU_0207/2V -> rcl:R-EU_0207/10
- SV2: device con-lstb:MA04-2 -> con-lsta:FE10-1
Connections:
- removed net +12V: IC1.CD+, IC4.CD+, SV2.1, SV2.2, SV2.3, SV2.4, X1GPA0-7-1.KL, X2-1.KL
- removed net GND: C1.2, C10.2, C11.2, C12.2, C13.2, C14.2, C15.2, C16.2, C19.1, C2.2, C20.2, C3.2, C4.2, C5.2, C6.2, C7.2, C8.2, C9.2, IC1.GND, IC2P.GND, IC3B.I, IC3B.O, IC3F.I, IC3F.O, IC3P.GND, IC4.GND, SV2.5, SV2.6, SV2.7, SV2.8, SV4.1, SV5.10, X2-2.KL, X2GPB0-7-1.KL
- removed net GPA1: IC1.O2, R18.2, R24.2, X1GPA0-7-8.KL
- removed net GPB0.: JP1.2, RN2.9, SV5.1
- removed net GPB1.: JP10.2, RN2.8, SV5.2
- removed net GPB2.: JP11.2, RN2.7, SV5.3
- removed net GPB3.: JP12.2, RN2.6, SV5.4
- removed net GPB4.: JP15.2, RN2.5, SV5.5
- removed net GPB5.: JP16.2, RN2.4, SV5.6
- removed net GPB6.: JP13.2, RN2.3, SV5.7
- removed net GPB7.: JP14.2, RN2.2, SV5.8
- removed net N$34: IC4.I1, JP1.3
- removed net N$35: C15.1, IC3C.I, R29.1
- removed net N$36: IC5F.O, JP2.3
- removed net N$38: IC5E.O, JP3.3
- removed net N$39: IC5D.O, JP4.3
- removed net N$40: IC5C.O, JP5.3
- removed net N$41: C16.1, IC3E.I, R32.1
- removed net N$42: IC3E.O, JP9.3
- removed net N$44: JP3.2, RN1.8, SV4.4
- removed net N$45: IC5B.O, JP6.3
- removed net N$46: IC5A.O, JP7.3
- removed net N$47: IC3C.O, JP8.3
- removed net N$48: JP5.2, RN1.6, SV4.6
- removed net N$49: IC1.I3, JP4.1
- removed net N$50: IC1.I1, JP2.1
- removed net N$51: IC1.I5, JP6.1
- removed net N$52: IC1.I4, JP5.1
- removed net N$53: IC1.I2, JP3.1
- removed net N$54: JP4.2, RN1.7, SV4.5
- removed net N$55: IC1.I7, JP8.1
- removed net N$56: IC1.I6, JP7.1
- removed net N$57: IC1.I8, JP9.1
- removed net N$58: JP6.2, RN1.5, SV4.7
- removed net N$59: JP7.2, RN1.4, SV4.8
- removed net N$60: JP8.2, RN1.3, SV4.9
- removed net N$61: JP9.2, RN1.2, SV4.10
- new net GPA1.: JP4.3, SV4.4
- new net IC1A0: ADR1.5, IC1.A0, R4.1
- new net IC1A1: ADR1.3, IC1.A1, R3.1
- new net IC1A2: ADR1.1, IC1.A2, R5.1
- new net INTA: IC1.INTA, JP1.7, JP1.8
- new net INTB: IC1.INTB, JP1.5, JP1.6
- new net N$17: JP5.1, SV1.3
- new net N$24: IC1.GPB7, JP18.2
- new net N$28: JP13.1, SV2.3
- new net RESETIC1: IC1.!RESET, R2.1
- new net SCL: IC1.SCL, JP1.11, JP1.12, R6.1
- new net SDA: IC1.SDA, JP1.10, JP1.9, R7.1
- new net VSS: ADR1.2, ADR1.4, ADR1.6, C2.2, IC1.VSS, JP1.1, JP1.2, JP2.2, LED1.A, S1.P1, SV1.1, SV2.10, SV4.1, SV5.10
- net GPA0: now also JP5.3, SV4.3; no longer IC1.O1, R17.2, R23.2, X1GPA0-7-9.KL
- net GPA2: now also JP3.3, SV4.5; no longer IC1.O3, R19.2, R25.2, X1GPA0-7-7.KL
- net GPA3: now also JP6.3, SV4.6; no longer IC1.O4, R20.2, R26.2, X1GPA0-7-6.KL
- net GPA4: now also JP7.3, SV4.7; no longer IC1.O5, R21.2, R27.2, X1GPA0-7-5.KL
- net GPA5: now also IC1.GPA5, JP8.2; no longer IC1.O6, R22.2, R28.2, X1GPA0-7-4.KL
- net GPA6: now also IC1.GPA6, JP9.2; no longer IC1.O7, R29.2, R31.2, X1GPA0-7-3.KL
- net GPA7: now also IC1.GPA7, JP10.2; no longer IC1.O8, R30.2, R32.2, X1GPA0-7-2.KL
- net GPB0: now also JP11.3, SV5.1; no longer IC4.O1, R10.2, R5.2, X2GPB0-7-9.KL
- net GPB1: now also JP12.3, SV5.2; no longer IC4.O2, R11.2, R4.2, X2GPB0-7-8.KL
- net GPB2: now also JP13.3, SV5.3; no longer IC4.O3, R33.2, R34.2, X2GPB0-7-7.KL
- net GPB3: now also JP14.3, SV5.4; no longer IC4.O4, R12.2, R16.2, X2GPB0-7-6.KL
- net GPB4: now also JP15.3, SV5.5; no longer IC4.O5, R14.2, R2.2, X2GPB0-7-5.KL
- net GPB5: now also JP16.3, SV5.6; no longer IC4.O6, R7.2, R8.2, X2GPB0-7-4.KL
- net GPB6: now also JP17.3, SV5.7; no longer IC4.O7, R13.2, R6.2, X2GPB0-7-3.KL
- net GPB7: now also JP18.3, SV5.8; no longer IC4.O8, R15.2, R9.2, X2GPB0-7-2.KL
- net N$1: now also LED1.C, R8.2; no longer IC2A.O, JP13.1
- net N$10: now also JP10.1, SV1.10; no longer IC4.I3, JP11.3
- net N$11: now also JP9.1, SV1.9; no longer C11.1, IC3D.I, R9.1
- net N$12: now also JP8.1, SV1.8; no longer JP2.2, RN1.9, SV4.3
- net N$13: now also JP7.1, SV1.7; no longer IC4.I4, JP12.3
- net N$14: now also JP6.1, SV1.6; no longer C2.1, IC5A.I, R22.1
- net N$15: now also JP3.1, SV1.5; no longer IC3D.O, JP14.1
- net N$16: now also JP4.1, SV1.4; no longer C14.1, IC5F.I, R17.1
- net N$18: now also IC1.GPB1, JP12.2; no longer IC2F.O, JP11.1
- net N$19: now also IC1.GPB2, JP13.2; no longer IC3A.O, JP12.1
- net N$2: now also JP9.3, SV4.9; no longer C7.1, IC2F.I, R33.1
- net N$20: now also IC1.GPB3, JP14.2; no longer IC2B.O, JP15.1
- net N$21: now also IC1.GPB4, JP15.2; no longer IC2C.O, JP16.1
- net N$22: now also IC1.GPB5, JP16.2; no longer IC4.I5, JP15.3
- net N$23: now also IC1.GPB6, JP17.2; no longer C13.1, IC5E.I, R18.1
- net N$25: now also JP11.1, SV2.1; no longer IC4.I6, JP16.3
- net N$26: now also IC1.GPB0, JP11.2; no longer IC4.I7, JP13.3
- net N$27: now also JP12.1, SV2.2; no longer IC4.I8, JP14.3
- net N$29: now also JP14.1, SV2.4; no longer C12.1, IC5D.I, R19.1
- net N$3: now also JP8.3, SV4.8; no longer IC2E.O, JP10.1
- net N$30: now also JP15.1, SV2.5; no longer IC2D.O, JP1.1
- net N$31: now also JP16.1, SV2.6; no longer C10.1, IC5C.I, R20.1
- net N$32: now also JP17.1, SV2.7; no longer C9.1, IC5B.I, R21.1
- net N$33: now also JP18.1, SV2.8; no longer IC4.I2, JP10.3
- net N$4: now also IC1.GPA4, JP7.2; no longer C1.1, IC2A.I, R6.1
- net N$5: now also IC1.GPA3, JP6.2; no longer C6.1, IC2E.I, R4.1
- net N$6: now also IC1.GPA2, JP3.2; no longer C5.1, IC2D.I, R5.1
- net N$7: now also IC1.GPA1, JP4.2; no longer C4.1, IC2C.I, R7.1
- net N$8: now also JP10.3, SV4.10; no longer C3.1, IC2B.I, R2.1
- net N$9: now also IC1.GPA0, JP5.2; no longer C8.1, IC3A.I, R12.1
- net VDD: now also C2.1, IC1.VDD, JP1.3, JP1.4, JP2.1, R2.2, R3.2, R4.2, R5.2, R6.2, R7.2, S1.S1, SV1.2, SV2.9; no longer C19.2, C20.1, IC2P.VCC, IC3P.VCC, R10.1, R11.1, R13.1, R14.1, R15.1, R16.1, R23.1, R24.1, R25.1, R26.1, R27.1, R28.1, R30.1, R31.1, R34.1, RN1.1, RN2.1
Other:
- moved on the sheet: C2, JP10, JP11, JP12, JP13, JP14, JP15, JP16, R2, R4, R5, R6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
