File: MCP23017_Aufsatz/MCP23017_Aufsatz_Verzweiger_V1.brd (EAGLE design)
At the start: 49.2 x 80 mm, 34 parts, among them IC1 MCP23017SP

Commit message: MCPAufsatzVerzweigerV1
Parts:
- moved C2 9.92 mm to (30.5, 49.5), turned to 90 degrees
Routing:
- net N$25: track 0.00 -> 14.7 mm
- net N$27: track 0.00 -> 13.6 mm
- net N$28: track 0.00 -> 13.0 mm
- net N$29: track 0.00 -> 12.5 mm
- net GPB5: track 0.00 -> 9.70 mm
- net N$18: track 0.00 -> 9.64 mm
- net GPB0: track 0.00 -> 8.67 mm
- net GPB4: track 0.00 -> 8.67 mm
- net GPB2: track 0.00 -> 8.48 mm
- net GPB1: track 0.00 -> 8.15 mm
- net GPB3: track 0.00 -> 8.15 mm
- net N$26: track 8.67 -> 10.7 mm
- net N$24: track 13.8 -> 14.7 mm
- net N$23: track 9.72 -> 10.5 mm
Other:
- board text added: "MCP23017Aufsatz Verzweiger (universal) Version V1"
- board text removed: "MCP23017Aufsatz (universal) Version V2"

Commit message: Aktuallisiert
Parts:
- turned JP5 to 0 degrees
Routing:
- net GPA0: track 19.8 -> 12.0 mm
- net N$17: track 8.45 -> 13.5 mm
- net VDD: track 140.2 -> 143.3 mm
- net N$11: track 15.1 -> 12.2 mm
- net SDA: track 20.1 -> 22.6 mm
- net GPB7: track 11.5 -> 13.0 mm
- net GPA5: track 8.95 -> 7.84 mm
